Commit message: fixed urdf, dice detection
Co-authored-by: Bela Ceniceros <bceni@users.noreply.github.com>

File: snakes_and_ladders/urdf/fourdof.urdf (robot description, URDF)
Before this commit: robot fourdof, 12 links, 11 joints
Links:
- added link gripper; visual mesh filename=package://snakes_and_ladders/meshes/Gripper_Part.STL scale=0.001 0.001 0.001
- link lbracket: geometry visual mesh filename=package://snakes_and_ladders/meshes/lower_bracket_improved_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 scale=0.001 0.001 0.001
Joints:
- added joint revolve: type fixed, parent gripper, child tip, origin xyz=0.05 0.1 0.025 rpy=0 0 0
- joint elbow: origin xyz=0 0 0.0311 rpy=0 0 0 -> xyz=0 0 0.01655 rpy=0 0 0
- joint gripper: child tip -> gripper; origin xyz=0.3450 0.00285 0.005 rpy=-1.5708 -1.5708 -1.5708 -> xyz=-0.0075 -0.0175 -0.055 rpy=-1.5708 -1.5708 -1.5708
- joint lbracket: origin xyz=0.0445 -0.017 0.1025 rpy=0 -1.5708 -1.5708 -> xyz=-0.038 0.02 0.113 rpy=0 -1.5708 1.5708
- joint upperarm: origin xyz=0.3850 -0.0025 0.0057 rpy=0 0 0 -> xyz=0.3850 -0.0025 0.0251 rpy=0 0 0
- joint wrist: origin xyz=0 0 0.0311 rpy=1.5708 -1.5708 0 -> xyz=0 0 -0.0321 rpy=3.14 1.5708 0
- joint wrist_rot: origin xyz=0.350 0  0.02 rpy=0 0 3.14 -> xyz=0.350 0  -0.01655 rpy=0 0 -3.14

Commit message: moving to player pieces success
Co-authored-by: Bela Ceniceros <bceni@users.noreply.github.com>
Co-authored-by: Brandon Frederick <brandon@caltech.edu>

File: snakes_and_ladders/urdf/fourdof.urdf (robot description, URDF)
Before this commit: robot fourdof, 13 links, 12 joints
Joints:
- joint revolve: origin xyz=0.05 0.1 0.025 rpy=0 0 0 -> xyz=0.05 0.15 0.025 rpy=0 0 0

Commit message: better position control

File: snakes_and_ladders/urdf/fourdof.urdf (robot description, URDF)
Before this commit: robot fourdof, 13 links, 12 joints
Joints:
- joint revolve: origin xyz=0.05 0.15 0.025 rpy=0 0 0 -> xyz=0.070 0.132 0.040 rpy=0 0 0

Commit message: updated trajectory to not hit the pieces and updated board game map to account for orientation
Co-authored-by: Bela Ceniceros <bceni@users.noreply.github.com>

File: snakes_and_ladders/urdf/fourdof.urdf (robot description, URDF)
Before this commit: robot fourdof, 13 links, 12 joints
Joints:
- joint revolve: origin xyz=0.070 0.132 0.040 rpy=0 0 0 -> xyz=0.070 0.132 0.04 rpy=0 0 0

Commit message: incorporated board game positions into movement

File: snakes_and_ladders/urdf/fourdof.urdf (robot description, URDF)
Before this commit: robot fourdof, 13 links, 12 joints
Joints:
- joint revolve: origin xyz=0.070 0.132 0.04 rpy=0 0 0 -> xyz=0.070 0.132 0.03 rpy=0 0 0

Commit message: Work on URDF

File: snakes_and_ladders/urdf/fourdof.urdf (robot description, URDF)
Before this commit: robot fourdof, 13 links, 12 joints
Links:
- link baseplate: geometry visual box size=0.1575 0.1175 0.0125
Joints:
- joint baseplate: origin xyz=0 0 0.0230 rpy=0 0 0 -> xyz=0 0.04 0.0125 rpy=0 0 0
- joint lbracket: origin xyz=-0.038 0.02 0.113 rpy=0 -1.5708 1.5708 -> xyz=-0.0385 0.037 0.1125 rpy=0 -1.5708 1.5708
- joint placement: origin xyz=0.748 0.01 0.0 rpy=0 0 0 -> xyz=0.0 0.0 0.0 rpy=0 0 0
- joint shoulder: origin xyz=0 0 0.03225 rpy=-3.14159 0 0.02 -> xyz=0 0 0.0451 rpy=-3.14159 0 0

Commit message: Work on precision and URDF
Co-authored-by: Bela Ceniceros <bceni@users.noreply.github.com>

File: snakes_and_ladders/urdf/fourdof.urdf (robot description, URDF)
Before this commit: robot fourdof, 13 links, 12 joints
Links:
- link lowerbracket: geometry visual mesh filename=package://snakes_and_ladders/meshes/l_bracket_gripper_0015.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 scale=0.001 0.001 0.001
Joints:
- joint elbow: origin xyz=0 0 0.01655 rpy=0 0 0 -> xyz=0 0 0.0311 rpy=0 0 0
- joint gripper: origin xyz=-0.0075 -0.0175 -0.055 rpy=-1.5708 -1.5708 -1.5708 -> xyz=0.0615 -0.0475 0 rpy=-1.5708 -1.5708 -1.5708
- joint placement: origin xyz=0.0 0.0 0.0 rpy=0 0 0 -> xyz=0.752 0.0 0.0 rpy=0 0 0
- joint revolve: origin xyz=0.070 0.132 0.03 rpy=0 0 0 -> xyz=0 0.127 0 rpy=0 0 0
- joint upperarm: origin xyz=0.3850 -0.0025 0.0251 rpy=0 0 0 -> xyz=0.3850 0 0 rpy=0 0 0
- joint wrist: origin xyz=0 0 -0.0321 rpy=3.14 1.5708 0 -> xyz=0 0 -0.0311 rpy=3.14159 1.5708 0
- joint wrist_rot: origin xyz=0.350 0  -0.01655 rpy=0 0 -3.14 -> xyz=0.325 0 0 rpy=0 0 -3.14159

Commit message: urdf changes, added blue player piece Co-authored-by: Bela Ceniceros <bceni@users.noreply.github.com> Co-authored-by: Brandon Frederick <brandon@caltech.edu>

File: snakes_and_ladders/urdf/fourdof.urdf (robot description, URDF)
Before this commit: robot fourdof, 13 links, 12 joints
Joints:
- joint placement: origin xyz=0.752 0.0 0.0 rpy=0 0 0 -> xyz=0.752 -0.01 0 rpy=0 0 0
- joint revolve: origin xyz=0 0.127 0 rpy=0 0 0 -> xyz=0 0.122 0 rpy=0 0 0
- joint shoulder: origin xyz=0 0 0.0451 rpy=-3.14159 0 0 -> xyz=0 0 0.0401 rpy=-3.14159 0 0
- joint wrist_rot: origin xyz=0.325 0 0 rpy=0 0 -3.14159 -> xyz=0.330 0 0 rpy=0 0 -3.14159

Commit message: updated urdf and improved cheating detection to not account for the board moving Co-authored-by: Bela Ceniceros <bceni@users.noreply.github.com> Co-authored-by: Brandon Frederick <brandon@caltech.edu>

File: snakes_and_ladders/urdf/fourdof.urdf (robot description, URDF)
Before this commit: robot fourdof, 13 links, 12 joints
Joints:
- joint upperarm: origin xyz=0.3850 0 0 rpy=0 0 0 -> xyz=0.3950 0 0 rpy=0 0 0
